Commit message: feat: add ackermann navigation, updated maps, and improved scripts
- Add Nav2 navigation stack with ackermann behavior tree and params
- Add cmd_vel_bridge and load_controllers scripts for ackermann control
- Add ackermann_map and real_map fixes (big/small) with SDF world
- Add third-party gazebo_ackermann_steering_vehicle package
- Add URDF model, map_to_sdf tool, diagnose/view scripts
- Add real-robot control plan and底盘485通信协议 documentation
- Update launch files, SLAM config, teleop scripts
- Remove outdated implementation/simulation plan docs
- Add CLAUDE.md to .gitignore (contains credentials)

File: models/ackermann/ackermann.xacro (robot description, xacro)
@@ -5,5 +5,5 @@
   <xacro:property name="body_width" value="0.6"/>
   <xacro:property name="body_height" value="0.4"/>
-  <xacro:property name="body_density" value="350.0"/>
+  <xacro:property name="body_density" value="150.0"/>
   <xacro:property name="wheel_radius" value="0.16"/>
   <xacro:property name="wheel_width" value="0.08"/>
@@ -11,7 +11,7 @@
   <xacro:property name="max_steering_angle" value="0.5236"/>
   <xacro:property name="max_steering_angular_velocity" value="1.570796"/>
-  <xacro:property name="max_steering_effort" value="50.0"/>
+  <xacro:property name="max_steering_effort" value="100.0"/>
   <xacro:property name="max_velocity" value="1.4"/>
-  <xacro:property name="max_effort" value="50.0"/>
+  <xacro:property name="max_effort" value="100.0"/>
   <xacro:property name="PI" value="3.14159265"/>
   <!-- Derived properties -->
@@ -85,4 +85,14 @@
       </material>
     </visual>
+    <!-- Rotation marker stripe (visual only) -->
+    <visual>
+      <origin xyz="${wheel_radius} 0 0" rpy="0 1.570795 0"/>
+      <geometry>
+        <box size="${wheel_width * 0.8} ${wheel_radius * 0.3} ${wheel_radius * 0.15}"/>
+      </geometry>
+      <material name="stripe_material_fl">
+        <color rgba="1.0 0.0 0.0 1.0"/>
+      </material>
+    </visual>
     <collision>
       <origin xyz="0 0 0" rpy="1.570795 0 0"/>
@@ -131,4 +141,14 @@
       </material>
     </visual>
+    <!-- Rotation marker stripe (visual only) -->
+    <visual>
+      <origin xyz="${wheel_radius} 0 0" rpy="0 1.570795 0"/>
+      <geometry>
+        <box size="${wheel_width * 0.8} ${wheel_radius * 0.3} ${wheel_radius * 0.15}"/>
+      </geometry>
+      <material name="stripe_material_fr">
+        <color rgba="1.0 0.0 0.0 1.0"/>
+      </material>
+    </visual>
     <collision>
       <origin xyz="0 0 0" rpy="1.570795 0 0"/>
@@ -154,4 +174,14 @@
       </material>
     </visual>
+    <!-- Rotation marker stripe (visual only) -->
+    <visual>
+      <origin xyz="${wheel_radius} 0 0" rpy="0 1.570795 0"/>
+      <geometry>
+        <box size="${wheel_width * 0.8} ${wheel_radius * 0.3} ${wheel_radius * 0.15}"/>
+      </geometry>
+      <material name="stripe_material_rl">
+        <color rgba="1.0 0.0 0.0 1.0"/>
+      </material>
+    </visual>
     <collision>
       <origin xyz="0 0 0" rpy="1.570795 0 0"/>
@@ -175,4 +205,14 @@
       <material name="wheel_material">
         <color rgba="0.0 0.0 0.0 1.0"/>
+      </material>
+    </visual>
+    <!-- Rotation marker stripe (visual only) -->
+    <visual>
+      <origin xyz="${wheel_radius} 0 0" rpy="0 1.570795 0"/>
+      <geometry>
+        <box size="${wheel_width * 0.8} ${wheel_radius * 0.3} ${wheel_radius * 0.15}"/>
+      </geometry>
+      <material name="stripe_material_rr">
+        <color rgba="1.0 0.0 0.0 1.0"/>
       </material>
     </visual>
@@ -197,5 +237,5 @@
     <axis xyz="0 0 1"/>
     <limit effort="${max_steering_effort}" lower="${-max_steering_angle}" upper="${max_steering_angle}" velocity="${max_steering_angular_velocity}"/>
-    <dynamics damping="0.1" friction="0.1"/>
+    <dynamics damping="0.01" friction="0.01"/>
   </joint>
   <!-- Front Left Wheel Joint (passive, Y-axis) -->
@@ -206,5 +246,5 @@
     <axis xyz="0 1 0"/>
     <limit effort="${max_effort}" velocity="${max_wheel_angular_velocity}"/>
-    <dynamics damping="0.1" friction="0.1"/>
+    <dynamics damping="0.01" friction="0.01"/>
   </joint>
   <!-- Front Right Steering Joint (position controlled, Z-axis) -->
@@ -215,5 +255,5 @@
     <axis xyz="0 0 1"/>
     <limit effort="${max_steering_effort}" lower="${-max_steering_angle}" upper="${max_steering_angle}" velocity="${max_steering_angular_velocity}"/>
-    <dynamics damping="0.1" friction="0.1"/>
+    <dynamics damping="0.01" friction="0.01"/>
   </joint>
   <!-- Front Right Wheel Joint (passive, Y-axis) -->
@@ -224,5 +264,5 @@
     <axis xyz="0 1 0"/>
     <limit effort="${max_effort}" velocity="${max_wheel_angular_velocity}"/>
-    <dynamics damping="0.1" friction="0.1"/>
+    <dynamics damping="0.01" friction="0.01"/>
   </joint>
   <!-- Rear Left Wheel Joint (velocity controlled, Y-axis) -->
@@ -233,5 +273,5 @@
     <axis xyz="0 1 0"/>
     <limit effort="${max_effort}" velocity="${max_wheel_angular_velocity}"/>
-    <dynamics damping="0.1" friction="0.1"/>
+    <dynamics damping="0.01" friction="0.01"/>
   </joint>
   <!-- Rear Right Wheel Joint (velocity controlled, Y-axis) -->
@@ -242,5 +282,5 @@
     <axis xyz="0 1 0"/>
     <limit effort="${max_effort}" velocity="${max_wheel_angular_velocity}"/>
-    <dynamics damping="0.1" friction="0.1"/>
+    <dynamics damping="0.01" friction="0.01"/>
   </joint>
   <!-- ========== Gazebo Surface Friction ========== -->
@@ -321,7 +361,4 @@
       <parameters>$(find ackermann_control)/config/gz_ros2_control.yaml</parameters>
     </plugin>
-    <plugin filename="gz-sim-sensors-system" name="gz::sim::systems::Sensors">
-      <render_engine>ogre2</render_engine>
-    </plugin>
     <plugin filename="gz-sim-imu-system" name="gz::sim::systems::Imu">
     </plugin>
@@ -344,5 +381,5 @@
         <scan>
           <horizontal>
-            <samples>3600</samples>
+            <samples>3200</samples>
             <resolution>1</resolution>
             <min_angle>0.0</min_angle>
@@ -352,5 +389,5 @@
         <range>
           <min>0.15</min>
-          <max>16.0</max>
+          <max>18.0</max>
         </range>
       </lidar>
