Commit message: feat: add auto-exploration, lidar_slam_nodes package, and reorganize scripts
- Add m-explore-ros2 and explore_lite for autonomous exploration
- Add frontier_explorer, scan_range_filter, map_saver_watcher nodes
- Add aws-robomaker-small-warehouse-world submodule
- Reorganize scripts into check/launch/tools subdirectories
- Add exploration launch and config files (rviz, nav2 params)
- Tune EKF and SLAM toolbox parameters
- Add param-tuning notes doc

Co-Authored-By: Claude Opus 4.7 <noreply@anthropic.com>

File: models/ackermann/ackermann.urdf (robot description, URDF)
Before this commit: robot ackermann_robot, 5 links, 4 joints
Links:
- removed link chassis
- removed link front_left_wheel
- removed link front_right_wheel
- removed link rear_left_wheel
- removed link rear_right_wheel
- added link body_link, mass 32.4; collision box size=0.9 0.6 0.4; visual box size=0.9 0.6 0.4
- added link front_left_steering_link, mass 0.01; collision cylinder length=0.001 radius=0.01; visual cylinder length=0.001 radius=0.01
- added link front_left_wheel_link, mass 5.790583572480001; collision cylinder length=0.08 radius=0.16; visual box size=0.064 0.048 0.024
- added link front_right_steering_link, mass 0.01; collision cylinder length=0.001 radius=0.01; visual cylinder length=0.001 radius=0.01
- added link front_right_wheel_link, mass 5.790583572480001; collision cylinder length=0.08 radius=0.16; visual box size=0.064 0.048 0.024
- added link rear_left_wheel_link, mass 5.790583572480001; collision cylinder length=0.08 radius=0.16; visual box size=0.064 0.048 0.024
- added link rear_right_wheel_link, mass 5.790583572480001; collision cylinder length=0.08 radius=0.16; visual box size=0.064 0.048 0.024
Joints:
- removed joint front_left_steering
- removed joint front_right_steering
- added joint front_left_steering_joint: type revolute, parent body_link, child front_left_steering_link, origin xyz=0.29000000000000004 0.33999999999999997 -0.08 rpy=0 0 0, axis 0 0 1, limit lower=-0.5236 upper=0.5236 effort=100.0 velocity=1.570796
- added joint front_left_wheel_joint: type continuous, parent front_left_steering_link, child front_left_wheel_link, origin xyz=0 0 0 rpy=0 0 0, axis 0 1 0, limit effort=100.0 velocity=8.75
- added joint front_right_steering_joint: type revolute, parent body_link, child front_right_steering_link, origin xyz=0.29000000000000004 -0.33999999999999997 -0.08 rpy=0 0 0, axis 0 0 1, limit lower=-0.5236 upper=0.5236 effort=100.0 velocity=1.570796
- added joint front_right_wheel_joint: type continuous, parent front_right_steering_link, child front_right_wheel_link, origin xyz=0 0 0 rpy=0 0 0, axis 0 1 0, limit effort=100.0 velocity=8.75
- joint rear_left_wheel_joint: child rear_left_wheel -> rear_left_wheel_link; limit (none) -> effort=100.0 velocity=8.75; origin xyz=-0.14 0.1 0 rpy=0 0 0 -> xyz=-0.29000000000000004 0.33999999999999997 -0.08 rpy=0 0 0; parent chassis -> body_link
- joint rear_right_wheel_joint: child rear_right_wheel -> rear_right_wheel_link; limit (none) -> effort=100.0 velocity=8.75; origin xyz=-0.14 -0.1 0 rpy=0 0 0 -> xyz=-0.29000000000000004 -0.33999999999999997 -0.08 rpy=0 0 0; parent chassis -> body_link

File: models/ackermann/ackermann.xacro (robot description, xacro)
@@ -36,5 +36,5 @@
       </geometry>
       <material name="body_material">
-        <color rgba="0.25 0.25 0.25 1.0"/>
+        <color rgba="0.5 0.0 0.5 1.0"/>
       </material>
     </visual>
@@ -70,5 +70,5 @@
     <inertial>
       <mass value="0.01"/>
-      <inertia ixx="0.0" ixy="0.0" ixz="0.0" iyy="0.0" iyz="0.0" izz="0.0"/>
+      <inertia ixx="1e-6" ixy="0.0" ixz="0.0" iyy="1e-6" iyz="0.0" izz="1e-6"/>
       <origin xyz="0 0 0" rpy="0 0 0"/>
     </inertial>
@@ -126,5 +126,5 @@
     <inertial>
       <mass value="0.01"/>
-      <inertia ixx="0.0" ixy="0.0" ixz="0.0" iyy="0.0" iyz="0.0" izz="0.0"/>
+      <inertia ixx="1e-6" ixy="0.0" ixz="0.0" iyy="1e-6" iyz="0.0" izz="1e-6"/>
       <origin xyz="0 0 0" rpy="0 0 0"/>
     </inertial>
@@ -286,4 +286,9 @@
   <!-- ========== Gazebo Surface Friction ========== -->
   <gazebo reference="body_link">
+    <material>
+      <ambient>0.5 0.0 0.5 1.0</ambient>
+      <diffuse>0.5 0.0 0.5 1.0</diffuse>
+      <specular>0.6 0.1 0.6 1.0</specular>
+    </material>
     <mu1>0.0001</mu1>
     <mu2>0.0001</mu2>
@@ -368,4 +373,5 @@
       <odom_topic>/odom</odom_topic>
       <dimensions>3</dimensions>
+      <publish_tf>false</publish_tf>
     </plugin>
   </gazebo>
@@ -375,10 +381,10 @@
     <sensor name="lidar" type="gpu_lidar">
       <pose>0 0 0.22 0 0 0</pose>
-      <topic>/scan</topic>
+      <topic>/scan_raw</topic>
       <update_rate>10</update_rate>
       <lidar>
         <scan>
           <horizontal>
-            <samples>3200</samples>
+            <samples>720</samples>
             <resolution>1</resolution>
             <min_angle>0.0</min_angle>
@@ -388,5 +394,5 @@
         <range>
           <min>0.15</min>
-          <max>18.0</max>
+          <max>16.0</max>
         </range>
       </lidar>

File: third-party/gazebo_ackermann_steering_vehicle/model/vehicle.xacro (robot description, xacro)
@@ -65,5 +65,5 @@
       </geometry>
       <material name="body_material">
-        <color rgba="0.25 0.25 0.25 1.0"/>
+        <color rgba="0.5 0.0 0.5 1.0"/>
       </material>
     </visual>
@@ -232,5 +232,5 @@
       </geometry>
       <material name="camera_stick_material">
-        <color rgba="0.25 0.25 0.25 1.0"/>
+        <color rgba="0.5 0.0 0.5 1.0"/>
       </material>
     </visual>
@@ -335,4 +335,9 @@
   <!-- Gazebo Parameters -->
   <gazebo reference="body_link">
+    <material>
+      <ambient>0.5 0.0 0.5 1.0</ambient>
+      <diffuse>0.5 0.0 0.5 1.0</diffuse>
+      <specular>0.6 0.1 0.6 1.0</specular>
+    </material>
     <mu1>0.0001</mu1>
     <mu2>0.0001</mu2>
